File: SensorBoard/Sensorboard.kicad_pcb (KiCad board)
At the start: 2 copper layers, 158.3 x 29.7 mm, 63 parts, among them J1 Conn_01x16_Pin, U1 LM339, U10 LM339, U2 CNY70, U3 CNY70, U4 CNY70, U5 CNY70, U6 CNY70, U7 CNY70, U8 CNY70

Commit message: Pinout Update
Routing:
- net +5V: track 276.7 -> 278.4 mm, vias 23 -> 24
