File: MainBoard/Main Board.kicad_pcb (KiCad board)
At the start: 2 copper layers, 120 x 107 mm, 66 parts, among them IC1 TLV61070ADBVR, J1 Motor, J2 Motor, J3 Row 2, J4 Row 2, J5 USB PowerOnly 6P, J8 FFC Connector, Q1 NMOS, Q2 NMOS, SW1 SS12D10G5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

Commit message: Updated Version
Routing:
- net +5V: track 55.9 -> 57.5 mm
- net /IR_6_D: track 8.83 -> 9.39 mm
- net /IR_6_A: track 28.4 -> 28.9 mm
