File: MainBoard/Main Board.kicad_pcb (KiCad board)
At the start: 2 copper layers, 120 x 107 mm, 73 parts, among them IC1 TLV61070ADBVR, J1 Motor, J2 Motor, J3 Row 2, J4 Row 2, J5 USB PowerOnly 6P, J6 Conn_01x02_Pin, J8 FFC Connector, Q1 NMOS, Q2 NMOS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

Commit message: Pinout Update
Parts:
- IC1: value TLV61070ADBVR -> TLV61046
- moved C13 6.04 mm to (124.4, 116.1), turned to -90 degrees
- moved R14 3.66 mm to (125.8, 116.6), turned to -90 degrees
- moved C14 1.25 mm to (127.0, 114.6)
- moved R13 1.25 mm to (125.8, 114.6)
Connections:
- IC1 pad 3: VBUS -> Net-(IC1-FB)
- IC1 pad 4: Net-(IC1-FB) -> VBUS
Routing:
- net Net-(IC1-FB): track 4.69 -> 13.7 mm
- net +5V: track 52.8 -> 51.0 mm
- net VBUS: track 83.7 -> 84.8 mm, vias 8 -> 7
- net GND: track 16.7 -> 15.7 mm, vias 187 -> 189
