File: MainBoard/Main Board.kicad_sch (KiCad schematic)
At the start: 66 parts, among them IC1 TLV61070ADBVR, J1 Motor, J2 Motor, J3 Row 2, J4 Row 2, J5 USB PowerOnly 6P, J8 FFC Connector, Q1 NMOS, Q2 NMOS, SW1 SS12D10G5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

Commit message: Finished MainBoard
Parts:
- added J6: Conn_01x02_Pin, Connector_PinHeader_2.54mm:PinHeader_1x02_P2.54mm_Vertical, symbol Connector:Conn_01x02_Pin
Connections:
- net GND: now also J6.2 (Pin_2); no longer U3.7
- net Vdrive: now also J6.1 (Pin_1)
- net at U2.1 (OD): now also U3.3; no longer U3.4
- net at U2.3 (OC): now also U3.1; no longer U3.5
- net at BT1.2 (-), C4.2, U2.6 (GND): now also U3.4; no longer U3.2, U3.3
Changed lines of the file:
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@@
 	)
 	(junction
-		(at 193.04 58.42)
+		(at 99.06 137.16)
 		(diameter 0)
 		(color 0 0 0 0)
@@
 	)
 	(junction
+		(at 193.04 39.37)
+		(diameter 0)
+		(color 0 0 0 0)
+	)
+	(junction
 		(at 165.1 133.35)
 		(diameter 0)
@@
 	)
 	(junction
-		(at 193.04 39.37)
-		(diameter 0)
-		(color 0 0 0 0)
-	)
-	(junction
 		(at 146.05 54.61)
 		(diameter 0)
@@
 	)
 	(junction
-		(at 193.04 40.64)
-		(diameter 0)
-		(color 0 0 0 0)
-	)
-	(junction
 		(at 20.32 93.98)
 		(diameter 0)
@@
 	(wire
 		(pts
-			(xy 193.04 39.37) (xy 200.66 39.37)
-		)
-		(stroke
-			(width 0)
-			(type default)
-		)
-	)
-	(wire
-		(pts
 			(xy 92.71 34.29) (xy 100.33 34.29)
 		)
@@
 	(wire
 		(pts
-			(xy 186.69 39.37) (xy 193.04 39.37)
-		)
-		(stroke
-			(width 0)
-			(type default)
-		)
-	)
-	(wire
-		(pts
 			(xy 151.13 158.75) (xy 151.13 162.56)
 		)
@@
 	(wire
 		(pts
-			(xy 193.04 39.37) (xy 193.04 40.64)
+			(xy 257.81 123.19) (xy 241.3 123.19)
 		)
 		(stroke
@@
 	(wire
 		(pts
-			(xy 257.81 123.19) (xy 241.3 123.19)
+			(xy 193.04 25.4) (xy 193.04 26.67)
 		)
 		(stroke
@@
 	(wire
 		(pts
-			(xy 193.04 25.4) (xy 193.04 26.67)
+			(xy 193.04 36.83) (xy 193.04 39.37)
 		)
 		(stroke
@@
 	(wire
 		(pts
-			(xy 193.04 58.42) (xy 194.31 58.42)
-		)
-		(stroke
-			(width 0)
-			(type default)
-		)
-	)
-	(wire
-		(pts
 			(xy 71.12 168.91) (xy 82.55 168.91)
 		)
@@
 	(wire
 		(pts
+			(xy 101.6 133.35) (xy 101.6 134.62)
+		)
+		(stroke
+			(width 0)
+			(type default)
+		)
+	)
+	(wire
+		(pts
 			(xy 88.9 106.68) (xy 88.9 107.95)
 		)
@@
 	(wire
 		(pts
+			(xy 99.06 137.16) (xy 102.87 137.16)
+		)
+		(stroke
+			(width 0)
+			(type default)
+		)
+	)
+	(wire
+		(pts
 			(xy 151.13 93.98) (xy 151.13 96.52)
 		)
@@
 	(wire
 		(pts
+			(xy 186.69 39.37) (xy 193.04 39.37)
+		)
+		(stroke
+			(width 0)
+			(type default)
+		)
+	)
+	(wire
+		(pts
 			(xy 69.85 137.16) (xy 69.85 138.43)
 		)
@@
 	(wire
 		(pts
-			(xy 193.04 58.42) (xy 193.04 60.96)
-		)
-		(stroke
-			(width 0)
-			(type default)
-		)
-	)
-	(wire
-		(pts
 			(xy 201.93 133.35) (xy 215.9 133.35)
 		)
@@
 	(wire
 		(pts
+			(xy 193.04 59.69) (xy 193.04 60.96)
+		)
+		(stroke
+			(width 0)
+			(type default)
+		)
+	)
+	(wire
+		(pts
 			(xy 95.25 168.91) (xy 106.68 168.91)
 		)
@@
 	(wire
 		(pts
-			(xy 193.04 36.83) (xy 193.04 39.37)
+			(xy 146.05 39.37) (xy 146.05 43.18)
 		)
 		(stroke
@@
 	(wire
 		(pts
-			(xy 146.05 39.37) (xy 146.05 43.18)
+			(xy 146.05 50.8) (xy 146.05 54.61)
 		)
 		(stroke
@@
 	(wire
 		(pts
-			(xy 146.05 50.8) (xy 146.05 54.61)
+			(xy 193.04 39.37) (xy 200.66 39.37)
 		)
 		(stroke
@@
 	(wire
 		(pts
-			(xy 193.04 40.64) (xy 194.31 40.64)
+			(xy 101.6 134.62) (xy 102.87 134.62)
 		)
 		(stroke
@@
 		(on_board yes)
 		(dnp no)
-		(fields_autoplaced yes)
 		(property "Reference" "R12"
-			(at 95.25 128.27 0)
+			(at 86.614 128.27 0)
 			(effects
 				(font
@@
 		)
 		(property "Value" "R"
-			(at 95.25 130.81 0)
+			(at 86.614 130.81 0)
 			(effects
 				(font
@@
 		(on_board yes)
 		(dnp no)
-		(fields_autoplaced yes)
 		(property "Reference" "C10"
 			(at 73.66 132.08 0)
@@
 			)
 		)
-		(pin "7"
-		)
-		(pin "2"
+		(pin "2,5"
 		)
-		(pin "1,8"
+		(pin "1"
 		)
 		(pin "4"
 		)
-		(pin "5"
-		)
 		(pin "3"
 		)
@@
 					(unit 1)
 				)
+			)
+		)
+	)
+	(symbol
+		(lib_id "Connector:Conn_01x02_Pin")
+		(at 107.95 134.62 0)
+		(mirror y)
+		(unit 1)
+		(exclude_from_sim no)
+		(in_bom yes)
+		(on_board yes)
+		(dnp no)
+		(property "Reference" "J6"
+			(at 109.22 136.144 0)
+			(effects
+				(font
+					(size 1.27 1.27)
+				)
+				(justify right)
+			)
+		)
+		(property "Value" "Conn_01x02_Pin"
+			(at 101.6 129.286 0)
+			(effects
+				(font
+					(size 1.27 1.27)
+				)
+				(justify right)
+				(hide yes)
+			)
+		)
+		(property "Footprint" "Connector_PinHeader_2.54mm:PinHeader_1x02_P2.54mm_Vertical"
+			(at 107.95 134.62 0)
+			(effects
+				(font
+					(size 1.27 1.27)
+				)
+				(hide yes)
+			)
+		)
+		(property "Datasheet" "~"
+			(at 107.95 134.62 0)
+			(effects
+				(font
+					(size 1.27 1.27)
+				)
+				(hide yes)
+			)
+		)
+		(property "Description" "Generic connector, single row, 01x02, script generated"
+			(at 107.95 134.62 0)
+			(effects
+				(font
+					(size 1.27 1.27)
+				)
+				(hide yes)
+			)
+		)
+		(pin "2"
+		)
+		(pin "1"
+		)
+		(instances
+			(project ""
+				(path "/d71fd82d-c528-433b-94ee-bbc6a2a196b5"
+					(reference "J6")
+					(unit 1)
+				)
+			)
+		)
+	)
+	(symbol
+		(lib_id "power:Vdrive")
+		(at 101.6 133.35 0)
+		(unit 1)
+		(exclude_from_sim no)
+		(in_bom yes)
+		(on_board yes)
+		(dnp no)
+		(fields_autoplaced yes)
+		(property "Reference" "#PWR013"
+			(at 96.52 137.16 0)
+			(effects
+				(font
+					(size 1.27 1.27)
+				)
+				(hide yes)
+			)
+		)
+		(property "Value" "Vdrive"
+			(at 101.6 128.27 0)
+			(effects
+				(font
+					(size 1.27 1.27)
+				)
+			)
+		)
+		(property "Footprint" ""
+			(at 101.6 133.35 0)
+			(effects
+				(font
+					(size 1.27 1.27)
+				)
+				(hide yes)
+			)
+		)
+		(property "Datasheet" ""
+			(at 101.6 133.35 0)
+			(effects
+				(font
+					(size 1.27 1.27)
+				)
+				(hide yes)
+			)
+		)
+		(property "Description" ""
+			(at 101.6 133.35 0)
+			(effects
+				(font
+					(size 1.27 1.27)
+				)
+				(hide yes)
+			)
+		)
+		(pin "1"
+		)
+		(instances
+			(project "Main Board"
+				(path "/d71fd82d-c528-433b-94ee-bbc6a2a196b5"
+					(reference "#PWR013")
+					(unit 1)
+				)

Commit message: Pinout Update
Parts:
- IC1: value TLV61070ADBVR -> TLV61046
- R13: value 90k -> 53k
Connections:
- net VBUS: now also IC1.4 (EN); no longer IC1.3 (EN)
- net at C14.2, R13.2, R14.1: now also IC1.3 (FB); no longer IC1.4 (FB)
Changed lines of the file:
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@@
 		)
 	)
-	(text_box "R_{13} = R_{14} * V_{out} / V_{REF} - R_{14}\nV_{REF} = 500 mV"
+	(text_box "R_{13} = R_{14} * V_{out} / V_{REF} - R_{14}\nV_{REF} = 795 mV"
 		(exclude_from_sim no)
 		(at 71.12 158.75 0)
@@
 		(fields_autoplaced yes)
 		(property "Reference" "R13"
-			(at 73.66 173.99 0)
-			(effects
-				(font
-					(size 1.27 1.27)
-				)
-				(justify left)
-			)
-		)
-		(property "Value" "90k"
-			(at 73.66 176.53 0)
+			(at 73.66 173.9899 0)
+			(effects
+				(font
+					(size 1.27 1.27)
+				)
+				(justify left)
+			)
+		)
+		(property "Value" "53k"
+			(at 73.66 176.5299 0)
 			(effects
 				(font
@@
 			)
 		)
-		(property "Value" "TLV61070ADBVR"
+		(property "Value" "TLV61046"
 			(at 53.34 162.56 0)
 			(effects
