File: BoostBoard/BoostBoard.kicad_pcb (KiCad board)
At the start: 2 copper layers, 17 x 17 mm, 11 parts, among them J1 Conn_01x02_Pin, J2 Conn_01x02_Pin, U1 MIC2288YML

Commit message: Uploaded Cad Models and recent PCB
Other:
- outline, holes or cut-outs redrawn
Changed lines of the file:
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@@
 		(allow_soldermask_bridges_in_footprints no)
 		(pcbplotparams
-			(layerselection 0x00010fc_ffffffff)
+			(layerselection 0x00010f0_ffffffff)
 			(plot_on_all_layers_selection 0x0000000_00000000)
 			(disableapertmacros no)
@@
 			(outputformat 1)
 			(mirror no)
-			(drillshape 1)
+			(drillshape 0)
 			(scaleselection 1)
-			(outputdirectory "")
+			(outputdirectory "M:/Projects/IEEE Line Follower/Outputs/")
 		)
 	)
@@
 		)
 		(property "Value" "D_Schottky"
-			(at 0 2.6 360)
+			(at 0 2.6 0)
 			(layer "F.Fab")
 			(effects
@@
 		)
 		(fp_text user "${REFERENCE}"
-			(at 0 -2.5 360)
+			(at 0 -2.5 0)
 			(layer "F.Fab")
 			(effects
@@
 		)
 		(fp_text user "${REFERENCE}"
-			(at 0 0 360)
+			(at 0 0 0)
 			(layer "F.Fab")
 			(effects
@@
 		(sheetfile "BoostBoard.kicad_sch")
 		(attr smd)
-		(fp_rect
+		(fp_line
+			(start 2.25 -1.5)
+			(end 2.25 -0.975)
+			(stroke
+				(width 0.15)
+				(type default)
+			)
+			(layer "F.SilkS")
+		)
+		(fp_line
 			(start -2.25 -1.5)
+			(end 2.25 -1.5)
+			(stroke
+				(width 0.15)
+				(type default)
+			)
+			(layer "F.SilkS")
+		)
+		(fp_line
+			(start -2.25 -0.95)
+			(end -2.25 -1.5)
+			(stroke
+				(width 0.15)
+				(type default)
+			)
+			(layer "F.SilkS")
+		)
+		(fp_line
+			(start 2.25 1.15)
 			(end 2.25 1.7)
 			(stroke
-				(width 0.1)
+				(width 0.15)
 				(type default)
 			)
-			(fill none)
+			(layer "F.SilkS")
+		)
+		(fp_line
+			(start 2.25 1.7)
+			(end -2.25 1.7)
+			(stroke
+				(width 0.15)
+				(type default)
+			)
+			(layer "F.SilkS")
+		)
+		(fp_line
+			(start -2.25 1.7)
+			(end -2.25 1.175)
+			(stroke
+				(width 0.15)
+				(type default)
+			)
 			(layer "F.SilkS")
 		)
@@
 		)
 		(property "Value" "10u"
-			(at 0 1.43 360)
+			(at 0 1.43 0)
 			(layer "F.Fab")
 			(effects
@@
 		)
 		(fp_text user "${REFERENCE}"
-			(at 0 0 360)
+			(at 0 0 0)
 			(layer "F.Fab")
 			(effects
@@
 		(tags "capacitor")
 		(property "Reference" "C1"
-			(at -2.1 0 360)
+			(at -2.1 0 0)
 			(layer "F.SilkS")
 			(effects
@@
 		)
 		(property "Value" "10u"
-			(at 0 1.43 360)
+			(at 0 1.43 0)
 			(layer "F.Fab")
 			(effects
@@
 		)
 		(fp_text user "${REFERENCE}"
-			(at 0 0 360)
+			(at 0 0 0)
 			(layer "F.Fab")
 			(effects
@@
 		(tags "Through hole pin header THT 1x02 2.54mm single row")
 		(property "Reference" "J1"
-			(at -2.075 -3.54 360)
+			(at -2.075 -3.54 0)
 			(layer "B.SilkS")
 			(effects
@@
 		)
 		(property "Value" "Conn_01x02_Pin"
-			(at 0 -4.87 360)
+			(at 0 -4.87 0)
 			(layer "B.Fab")
 			(effects
@@
 		)
 		(fp_text user "${REFERENCE}"
-			(at 0 -1.27 360)
+			(at 0 -1.27 0)
 			(layer "B.Fab")
 			(effects
@@
 		)
 	)
-	(gr_rect
-		(start 110 90)
-		(end 127 107)
+	(gr_line
+		(start 126 107)
+		(end 111 107)
 		(stroke
 			(width 0.05)
 			(type default)
 		)
-		(fill none)
 		(layer "Edge.Cuts")
 	)
+	(gr_arc
+		(start 126 90)
+		(mid 126.707107 90.292893)
+		(end 127 91)
+		(stroke
+			(width 0.05)
+			(type default)
+		)
+		(layer "Edge.Cuts")
+	)
+	(gr_arc
+		(start 111 107)
+		(mid 110.292893 106.707107)
+		(end 110 106)
+		(stroke
+			(width 0.05)
+			(type default)
+		)
+		(layer "Edge.Cuts")
+	)
+	(gr_line
+		(start 111 90)
+		(end 126 90)
+		(stroke
+			(width 0.05)
+			(type default)
+		)
+		(layer "Edge.Cuts")
+	)
+	(gr_line
+		(start 110 106)
+		(end 110 91)
+		(stroke
+			(width 0.05)
+			(type default)
+		)
+		(layer "Edge.Cuts")
+	)
+	(gr_line
+		(start 127 91)
+		(end 127 106)
+		(stroke
+			(width 0.05)
+			(type default)
+		)
+		(layer "Edge.Cuts")
+	)
+	(gr_arc
+		(start 127 106)
+		(mid 126.707107 106.707107)
+		(end 126 107)
+		(stroke
+			(width 0.05)
+			(type default)
+		)
+		(layer "Edge.Cuts")
+	)
+	(gr_arc
+		(start 110 91)
+		(mid 110.292893 90.292893)
+		(end 111 90)
+		(stroke
+			(width 0.05)
+			(type default)
+		)
+		(layer "Edge.Cuts")
+	)
