File: BoostBoard/BoostBoard.kicad_sch (KiCad schematic)
At the start: 11 parts, among them J1 Conn_01x02_Pin, J2 Conn_01x02_Pin, U1 MIC2288YML

Commit message: Uploaded Cad Models and recent PCB
Changed lines of the file:
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@@
+		)
+	)
+	(text_box "Vout |	RT	|RB\n12	|	47k	|5.49k\n10	|	39k	|5.49k\n8	|	30k	|5.49k"
+		(exclude_from_sim no)
+		(at 100.33 111.76 0)
+		(size 24.13 10.16)
+		(stroke
+			(width 0)
+			(type default)
+		)
+		(fill
+			(type none)
+		)
+		(effects
+			(font
+				(size 1.27 1.27)
+			)
+			(justify left top)
 		)
 	)
