File: MainBoardV2/Main Boardv2.kicad_pcb (KiCad board)
At the start: 2 copper layers, 120 x 107 mm, 78 parts, among them IC1 TLV61046, J2 FFC Connector, J3 Motor, J4 Row 2, J5 Row 2, J6 Motor, J7 USB_C_Receptacle_USB2.0_16P, Q1 IRF540, Q2 IRF540, SW1 SS12D10G5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

Commit message: Uploaded Cad Models and recent PCB
Parts:
- removed C12, C13, C14, C6: 10u, Capacitor_SMD:C_0603_1608Metric
- removed D10, D9: LED, LED_SMD:LED_0603_1608Metric
- removed D6, D7: D_Schottky, Diode_SMD:D_SMA
- removed L1, L3: 10u, 0_Inductors:Murata_LQH43xxx
- removed R11, R17, R19, R20: 5.49k, Resistor_SMD:R_0603_1608Metric
- removed R16, R8: 30k, Resistor_SMD:R_0603_1608Metric
- removed U4, U5: ~, Package_TO_SOT_SMD:SOT-23-5_HandSoldering
- added J1: Conn_01x02_Pin, Connector_PinHeader_2.54mm:PinHeader_1x02_P2.54mm_Vertical, F.Cu at (109.2, 122.8)
- added J10: Conn_01x02_Pin, Connector_PinHeader_2.54mm:PinHeader_1x02_P2.54mm_Vertical, F.Cu at (191.3, 120.3)
- added J8: Conn_01x02_Pin, Connector_PinHeader_2.54mm:PinHeader_1x02_P2.54mm_Vertical, F.Cu at (95.4, 120.3)
- added J9: Conn_01x02_Pin, Connector_PinHeader_2.54mm:PinHeader_1x02_P2.54mm_Vertical, F.Cu at (205.0, 122.8)
- moved C8 221.1 mm to (189.5, 51.2)
- moved IC1 216.7 mm to (187.5, 54.1), turned to 90 degrees
- moved C9 213.1 mm to (188.3, 48.2)
- moved C10 211.3 mm to (186.1, 49.8), turned to 90 degrees
- moved C11 210.6 mm to (184.6, 49.8), turned to 90 degrees
- moved R15 210.2 mm to (188.3, 46.7), turned to 180 degrees
- moved R13 207.4 mm to (188.3, 49.7)
- moved L2 206.5 mm to (182.5, 54.3), turned to -90 degrees
- moved R4 9.14 mm to (113.9, 42.0), turned to 180 degrees
- moved R5 5.22 mm to (127.5, 45.0), turned to -90 degrees
- moved D1 0.60 mm to (123.9, 56.0)
- moved D2 0.60 mm to (125.4, 56.0)
- moved R6 0.60 mm to (123.9, 53.0)
- moved R7 0.60 mm to (125.4, 53.0)
Routing:
- net VBUS: track 0.00 -> 296.5 mm
- net Net-(BT1--): track 0.00 -> 166.4 mm, vias 0 -> 16
- net +5V: track 0.00 -> 156.9 mm, vias 0 -> 8
- net /PWM_R: track 0.00 -> 112.9 mm, vias 0 -> 2
- net /IR_3_A: track 0.00 -> 101.1 mm, vias 0 -> 1
- net Net-(BT1-+): track 0.00 -> 100.8 mm, vias 0 -> 4
- net /IR_4_A: track 0.00 -> 100.2 mm, vias 0 -> 1
- net /IR_6_A: track 0.00 -> 98.9 mm, vias 0 -> 1
- net /IR_2_A: track 0.00 -> 98.2 mm, vias 0 -> 1
- net /IR_5_A: track 0.00 -> 97.2 mm, vias 0 -> 1
- net /PWM_L: track 0.00 -> 88.9 mm, vias 0 -> 1
- net /IR_3_D: track 0.00 -> 82.2 mm, vias 0 -> 2
- net /IR_1_D: track 0.00 -> 79.8 mm, vias 0 -> 2
- net /IR_5_D: track 0.00 -> 77.9 mm, vias 0 -> 1
- net /IR_2_D: track 0.00 -> 77.0 mm, vias 0 -> 2
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- added copper zone on F.Cu, net +5V
- added copper zone on B.Cu, net GND
- added copper zone on F.Cu, net GND
- added copper zone on B.Cu, net Net-(BT1-+)
- added copper zone on F.Cu, net Net-(BT1-+)
- added copper zone on B.Cu, net Net-(BT1--)
- added copper zone on F.Cu, net Net-(BT1--)
- added copper zone on F.Cu, net Net-(IC1-SW)
- added copper zone on F.Cu, net VBUS
