File: MainBoardV2/Main Boardv2.kicad_sch (KiCad schematic)
At the start: 74 parts, among them IC1 TLV61046, J2 FFC Connector, J3 Motor, J4 Row 2, J5 Row 2, J6 Motor, J7 USB_C_Receptacle_USB2.0_16P, Q1 IRF540, Q2 IRF540, SW1 SS12D10G5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

Commit message: Uploaded Cad Models and recent PCB
Parts:
- removed C12, C13, C14, C6: 10u, Capacitor_SMD:C_0603_1608Metric, symbol Device:C
- removed D10, D9: LED, LED_SMD:LED_0603_1608Metric, symbol Device:LED
- removed D6, D7: D_Schottky, Diode_SMD:D_SMA, symbol Device:D_Schottky
- removed L1, L3: 10u, 0_Inductors:Murata_LQH43xxx, symbol Device:L
- removed R11, R17, R19, R20: 5.49k, Resistor_SMD:R_0603_1608Metric, symbol Device:R
- removed R16, R8: 30k, Resistor_SMD:R_0603_1608Metric, symbol Device:R
- removed U4, U5: ~, Package_TO_SOT_SMD:SOT-23-5_HandSoldering, symbol 0_Switching_Regulators:MIC2288
- added J1, J10, J8, J9: Conn_01x02_Pin, Connector_PinHeader_2.54mm:PinHeader_1x02_P2.54mm_Vertical, symbol Connector:Conn_01x02_Pin
Connections:
- net GND: now also J1.2 (Pin_2), J10.2 (Pin_2), J8.2 (Pin_2), J9.2 (Pin_2)
- net VBUS: now also J1.1 (Pin_1), J9.1 (Pin_1)
- net VMOTL: now also J10.1 (Pin_1)
- net VMOTR: now also J8.1 (Pin_1)
Other:
- note added: "Replacable Boost Board"
- note removed: "MIC2288YML"
