File: SensorBoardV2/SensorboardV2.kicad_sch (KiCad schematic)
At the start: 56 parts, among them J1 Conn_01x16_Pin, U1 LM339, U10 LM339, U2 CNY70, U3 CNY70, U4 CNY70, U5 CNY70, U6 CNY70, U7 CNY70, U8 CNY70

Commit message: Final Update
Connections:
- net IR_2_A: now also U1.6 (-); no longer U1.7 (+)
- net IR_6_A: now also U10.6 (-); no longer U10.7 (+)
- net at C7.1, RV6.2: now also U10.7 (+); no longer U10.6 (-)
- net at C2.1, RV2.2: now also U1.7 (+); no longer U1.6 (-)
Changed lines of the file:
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@@
 		(lib_id "Comparator:LM339")
 		(at 185.42 86.36 0)
+		(mirror x)
 		(unit 2)
 		(exclude_from_sim no)
@@
 		(on_board yes)
 		(dnp no)
-		(fields_autoplaced yes)
 		(property "Reference" "U10"
-			(at 185.42 76.2 0)
+			(at 185.42 96.52 0)
 			(effects
 				(font
@@
 		)
 		(property "Value" "LM339"
-			(at 185.42 78.74 0)
+			(at 185.42 93.98 0)
 			(effects
 				(font
@@
 		)
 		(property "Footprint" "Package_SO:SO-14_3.9x8.65mm_P1.27mm"
-			(at 184.15 83.82 0)
+			(at 184.15 88.9 0)
 			(effects
 				(font
@@
 		)
 		(property "Datasheet" "https://www.st.com/resource/en/datasheet/lm139.pdf"
-			(at 186.69 81.28 0)
+			(at 186.69 91.44 0)
 			(effects
 				(font
@@
 		(lib_id "Comparator:LM339")
 		(at 85.09 86.36 0)
+		(mirror x)
 		(unit 2)
 		(exclude_from_sim no)
@@
 		(on_board yes)
 		(dnp no)
-		(fields_autoplaced yes)
 		(property "Reference" "U1"
-			(at 85.09 76.2 0)
+			(at 85.09 96.52 0)
 			(effects
 				(font
@@
 		)
 		(property "Value" "LM339"
-			(at 85.09 78.74 0)
+			(at 85.09 93.98 0)
 			(effects
 				(font
@@
 		)
 		(property "Footprint" "Package_SO:SO-14_3.9x8.65mm_P1.27mm"
-			(at 83.82 83.82 0)
+			(at 83.82 88.9 0)
 			(effects
 				(font
@@
 		)
 		(property "Datasheet" "https://www.st.com/resource/en/datasheet/lm139.pdf"
-			(at 86.36 81.28 0)
-			(effects
-				(font
+			(at 86.36 91.44 0)
+			(effects
+				(font
